File: BenchBuddy/BenchBuddy.kicad_pcb (KiCad board)
At the start: 4 copper layers, 152.4 x 63.5 mm, 11 parts, among them K1 1461069-5, Q1 2N3904, U1 LTV-816S

Commit message: Pre layout
Parts:
- added 3 mm: VAL**, 3mm_NPTH, F.Cu at (73.8, 77.9)
- added 3 mm: VAL**, 3mm_NPTH, F.Cu at (73.9, 134.6)
- added 3 mm: VAL**, 3mm_NPTH, F.Cu at (213.2, 77.9)
- added 3 mm: VAL**, 3mm_NPTH, F.Cu at (219.2, 119.9)
- added ARD1: ARDUINOPINS, Arduino, F.Cu at (121.9, 109.7)
- added C1: C, SM0805, B.Cu at (141.4, 99.1)
- added C10: C, SM0805, B.Cu at (198.0, 88.1)
- added C11: C, SM0805, B.Cu at (141.9, 108.5)
- added C12: C, SM0805, B.Cu at (205.5, 96.0)
- added C13: C, SM1206, B.Cu at (61.8, 89.3)
- added C14: C, SM0805, B.Cu at (174.2, 147.2)
- added C15: C, SM0805, B.Cu at (185.2, 147.2)
- added C16: C, SM0805, B.Cu at (177.9, 147.2)
- added C17: C, SM0805, B.Cu at (181.5, 147.2)
- added C18: C, SM0805, B.Cu at (166.9, 147.2)
- added C19: C, SM0805, B.Cu at (159.4, 147.1)
- added C2: C, SM1206, F.Cu at (99.7, 117.3)
- added C20: C, SM0805, B.Cu at (188.9, 147.2)
- added C21: C, SM0805, B.Cu at (192.6, 147.2)
- added C22: C, SM0805, B.Cu at (170.6, 147.2)
- added C23: C, SM0805, B.Cu at (148.5, 147.2)
- added C24: C, SM0805, B.Cu at (193.3, 143.4)
- added C25: C, SM0805, B.Cu at (163.2, 147.2)
- added C3: C, SM1206, F.Cu at (99.7, 121.9)
- added C4: 1 uF, SM0805, B.Cu at (152.8, 116.3)
- added C5: 1 uF, SM0805, B.Cu at (155.7, 116.5)
- added C6: C, SM0805, B.Cu at (138.4, 103.0)
- added C7: C, SM0805, B.Cu at (145.5, 102.2)
- added C8: C, SM0805, F.Cu at (212.5, 103.8)
- added C9: C, SM0805, B.Cu at (177.5, 99.3)
- added D10: MMBD914-7F, SOT23_Diode, F.Cu at (161.6, 144.2)
- added D11: MMBD914-7F, SOT23_Diode, F.Cu at (158.2, 144.2)
- added D12: MMBD914-7F, SOT23_Diode, F.Cu at (171.5, 144.3)
- added D3: MMBD914-7F, SOT23_Diode, F.Cu at (148.3, 144.3)
- added D4: B4540WS-7, SOD-323, F.Cu at (152.4, 117.5)
- added D5: B130-13-F, SMA, F.Cu at (205.0, 84.0)
- added D6: MMBD914-7F, SOT23_Diode, F.Cu at (168.3, 144.3)
- added D7: MMBD914-7F, SOT23_Diode, F.Cu at (151.6, 144.2)
- added D8: MMBD914-7F, SOT23_Diode, F.Cu at (165.0, 144.2)
- added D9: MMBD914-7F, SOT23_Diode, F.Cu at (154.9, 144.3)
- added JP1: JUMPER, PIN_ARRAY_2X1, F.Cu at (143.4, 144.1)
- added L1: CM322522-220KL, SM1210L, B.Cu at (65.6, 89.4)
- added L2: CM322522-220KL, SM1210L, F.Cu at (91.3, 117.3)
- added L3: 22uH, NR4012, F.Cu at (160.9, 115.1)
- added L4: CM322522-220KL, SM1210L, F.Cu at (91.3, 121.8)
- added L5: INDUCTOR, SM0805, F.Cu at (209.7, 146.4)
- added P1: 24 Pin MiniFit JR, ATX_Header, F.Cu at (63.9, 82.8)
- added P2: CONN_3X2, pin_array_3x2, F.Cu at (164.5, 97.9)
- added P3: CONN_2, PIN_ARRAY_2X1, F.Cu at (135.3, 96.7)
- added P4: 12 Pin Terminal Block, 12_PinTB, F.Cu at (221.2, 114.9)
- added P5: 3 Pin Terminal Block, 3_PinTB, F.Cu at (220.7, 134.7)
- added Q2: DMN65D8L-7, SOT23GDS, F.Cu at (183.6, 93.3)
- added Q3: AOD476, DPAK2, F.Cu at (211.8, 95.8)
- added Q4: AOD476, DPAK2, F.Cu at (200.9, 95.7)
- added R10: R, SM0805_Blob, F.Cu at (141.3, 125.4)
- added R11: R, SM0805_Blob, F.Cu at (143.9, 125.5)
- added R12: R, SM0805_Blob, F.Cu at (114.1, 86.7)
- added R13: R, SM0805_Blob, F.Cu at (116.9, 86.7)
- added R14: R, SM0805_Blob, F.Cu at (119.4, 86.6)
- added R15: R, SM0805_Blob, F.Cu at (121.9, 86.7)
- added R16: R, SM0805_Blob, F.Cu at (124.4, 86.9)
- added R17: R, SM0805_Blob, F.Cu at (127.0, 86.9)
- added R18: R, SM0805_Blob, F.Cu at (131.1, 86.9)
- added R19: R, SM0805_Blob, F.Cu at (146.2, 86.9)
- added R20: R, SM0805_Blob, F.Cu at (149.0, 86.9)
- added R21: R, SM1206, B.Cu at (177.6, 98.5)
- added R22: R, SM1206, B.Cu at (174.2, 98.5)
- added R23: R, SM1206, B.Cu at (184.5, 98.4)
- added R24: R, SM1206, B.Cu at (181.0, 98.5)
- added R25: R, SM0805, F.Cu at (179.4, 92.6)
- added R26: R, SM0805, B.Cu at (171.8, 129.4)
- added R27: R, SM0805, B.Cu at (170.6, 98.6)
- added R28: R, SM0805, F.Cu at (82.4, 131.8)
- added R29: 15R, SM0805, B.Cu at (158.8, 116.3)
- added R30: 5k, EVUE3K, F.Cu at (196.3, 79.6)
- added R31: 715, SM0805, B.Cu at (182.4, 143.6)
- added R32: 715, SM0805, B.Cu at (155.8, 147.2)
- added R33: 5k, EVUE3K, F.Cu at (183.1, 79.6)
- added R36: R, SM0805, F.Cu at (179.6, 144.5)
- added R37: R, SM0805, F.Cu at (177.8, 144.5)
- added R38: R, SM0805, F.Cu at (176.0, 144.5)
- added R39: R, SM0805, F.Cu at (174.1, 144.5)
- added R40: R, SM0805, B.Cu at (198.5, 92.4)
- added R41: R, SM1206, B.Cu at (193.7, 96.8)
- added R42: R, SM0805, B.Cu at (170.7, 92.8)
- added R43: R, SM0805, B.Cu at (173.4, 92.7)
- added R44: R, SM0805, B.Cu at (176.0, 92.7)
- added R45: R, SM0805_Blob, F.Cu at (136.0, 86.7)
- added R46: R, SM0805_Blob, F.Cu at (138.7, 86.7)
- added R47: R, SM0805_Blob, F.Cu at (123.4, 125.5)
- added R48: R, SM0805_Blob, F.Cu at (126.1, 125.6)
- added R49: R, SM0805_Blob, F.Cu at (128.9, 125.6)
- added R50: 0, SM0805, B.Cu at (146.4, 96.5)
- added R51: 0, SM0805, B.Cu at (141.4, 94.6)
- added R52: R, SM0805_Blob, F.Cu at (141.4, 87.0)
- added R53: R, SM0805_Blob, F.Cu at (143.6, 86.7)
- added R54: R, SM0805, B.Cu at (152.2, 147.2)
- added R55: R, SM0805, B.Cu at (148.5, 149.0)
- added R56: R, SM0805, B.Cu at (152.1, 148.9)
- added R57: R, SM0805, B.Cu at (186.0, 143.4)
- added R7: R, SM0805_Blob, F.Cu at (131.6, 125.6)
- added R8: R, SM0805_Blob, F.Cu at (136.2, 125.5)
- added R9: R, SM0805_Blob, F.Cu at (138.8, 125.4)
- added SW1: Power Switch, BB_Switch, F.Cu at (117.2, 62.4)
- added TH1: MINISMDC050F-2, SM1812, B.Cu at (84.5, 91.3)
- added TH2: MINISMDC050F-2, SM1812, B.Cu at (65.5, 96.6)
- added TH3: MINISMDC050F-2, SM1812, B.Cu at (96.1, 125.3)
- added TH4: MINISMDC050F-2, SM1812, B.Cu at (83.7, 124.7)
- added TH5: MINISMDC050F-2, SM1812, F.Cu at (193.0, 91.2)
- added TP1: CONN_1, 1pin, F.Cu at (201.9, 146.1)
- added U11: MCP4801, SO8N, F.Cu at (141.6, 112.1)
- added U2: MCP3901, SSOP20, F.Cu at (141.3, 97.6)
- added U3: LMT84, SOT353, F.Cu at (215.8, 102.9)
- added U4: OPA4170, SO14N, F.Cu at (177.5, 99.2)
- added U5: AP5726, SOT23_6, F.Cu at (155.7, 116.3)
- added U6: LM317, TO220_VERT, F.Cu at (169.8, 77.4)
- added U7: LM337T, TO220_VERT, F.Cu at (157.5, 77.3)
- added U8: LM337T, TO220_VERT, F.Cu at (169.9, 87.8)
- added U9: LM317, TO220_VERT, F.Cu at (157.7, 87.7)
- moved U1 57.7 mm to (175.8, 133.4)
- moved R4 55.4 mm to (179.5, 129.1)
- moved R6 52.8 mm to (189.7, 143.6)
- moved R1 52.2 mm to (174.5, 129.4)
- moved R5 51.8 mm to (183.4, 129.0)
- moved K1 47.0 mm to (197.6, 129.2)
- moved D1 46.9 mm to (192.1, 129.3)
- moved Q1 46.9 mm to (194.8, 136.0)
- moved R2 46.9 mm to (187.4, 128.5)
- moved R3 46.9 mm to (194.8, 132.0)
- moved D2 45.4 mm to (189.2, 136.0)
Connections:
- K1 pad 1: (no net) -> /Relay/RELAY_COM
- K1 pad 3: (no net) -> /Relay/RELAY_NC
- K1 pad 4: (no net) -> /Relay/RELAY_NO
- R1 pad 1: GND -> /Arduino/RELAY-
- R2 pad 2: GND -> GND_RELAY
- R6 pad 2: GND -> GND_RELAY
Other:
- board size 152.4 x 63.5 mm -> 165.1 x 63.5 mm

Commit message: Pre layout 2
Parts:
- added C26: 10u, SM1210, F.Cu at (240.3, 123.1)
- added C27: 10u, SM1210, F.Cu at (239.3, 128.0)
- added C28: 10u, SM1210, F.Cu at (220.2, 141.7)
- added C29: 10u, SM1210, F.Cu at (220.8, 146.2)
- added C30: NoPop, SM0805, F.Cu at (241.7, 117.1)
- added C31: NoPop, SM0805, F.Cu at (249.6, 127.2)
- added R34: 0, SM0805, F.Cu at (246.0, 113.2)
- C1: value C -> 100PF
- C10, C11, C12, C6, C7, C8, C9: value C -> 1u
- C13, C14, C15, C16, C17, C2, C22, C23, C24, C25, C3: value C -> 10u
- C18, C19, C20, C21: value C -> .01u
- L5: value INDUCTOR -> 1u
- R1: value 500 -> 200
- R10, R11, R12, R13, R14, R15, R16, R17, R18, R19, R20, R45, R46, R47, R48, R49, R52, R53, R7, R8, R9: value R -> 0; footprint SM0805_Blob -> SM0805_SB
- R21, R22, R25, R27: value R -> 5K
- R23, R24: value R -> 200K
- R26, R28, R40: value R -> 0
- R36, R39: value R -> 1K
- R37, R38: value R -> 3K
- R41: value R -> 1
- R42: value R -> 10
- R43: value R -> 100
- R44: value R -> 1000
- R54, R57: value R -> 9.1K
- R55, R56: value R -> 1.3K
- U6, U9: value LM317 -> LM317T; footprint TO220_VERT -> TO220_BB
- U7, U8: footprint TO220_VERT -> TO220_BB
- moved U7 114.3 mm to (251.4, 142.7), turned to 0 degrees
- moved U9 97.2 mm to (237.6, 143.1), turned to 0 degrees
- moved U8 93.5 mm to (245.0, 143.4), turned to 0 degrees
- moved U6 91.3 mm to (230.7, 145.4), turned to 0 degrees
Connections:
- ARD1 pad 12: N-0000036 -> (no net)
- ARD1 pad 17: (no net) -> N-0000036
- C19 pad 1: N-00000128 (its old number) -> N-00000135
- C20 pad 1: N-00000130 -> N-00000134
- D11 pad 1: N-00000130 -> N-00000134
- D12 pad 1: N-00000128 (its old number) -> N-00000135
- D3 pad 1: /PowerAdjustmentMonitor/V-_ADJ -> -12V
- D3 pad 2: -12V -> /PowerAdjustmentMonitor/V-_ADJ
- D7 pad 1: FE_V- -> -12V
- D7 pad 2: -12V -> FE_V-
- Q2 pad S: AGND -> N-00000122
- Q4 pad 1: N-00000125 -> N-00000123
- R30 pad 1: N-00000128 (its old number) -> N-00000135
- R31 pad 1: N-00000128 (its old number) -> N-00000135
- R56 pad 1: N-00000130 -> N-00000134
- R57 pad 2: N-00000130 -> N-00000134
- U2 pad 10: (no net) -> AGND
- U2 pad 15: (no net) -> N-0000070
- U2 pad 16: (no net) -> N-0000071
- U2 pad 9: (no net) -> N-0000067
- U4 pad 6: /Arduino/CURR_MEAS -> N-00000126
- U4 pad 7: N-00000125 -> N-00000124
- U6 pad 1: +12V -> N-00000135
- U6 pad 2: N-00000128 (its old number) -> /PowerAdjustmentMonitor/V+_ADJ
- U6 pad 3: /PowerAdjustmentMonitor/V+_ADJ -> +12V
- U9 pad 1: +12V -> N-00000134
- U9 pad 2: N-00000130 -> FE_V+
- U9 pad 3: FE_V+ -> +12V
Other:
- net class Default: clearance 0.254 -> 0.1524
- rule pad_to_mask_clearance: 0.0508 -> 0.0254
- rule trace_clearance: 0.254 -> 0.1524
