File: BenchBuddy/BenchBuddy.sch (KiCad schematic (older format))
At the start: 0 parts

Commit message: Week3 part 1
Changed lines of the file:
@@
 $Descr A4 11693 8268
 encoding utf-8
-Sheet 1 8
+Sheet 1 9
 Title ""
-Date "1 feb 2014"
+Date "5 mar 2014"
 Rev ""
 Comp ""
@@
 $EndDescr
 $Sheet
-S 3600 3200 1400 3450
+S 2750 3300 1400 3450
 U 52ED6BE1
 F0 "Arduino" 50
 F1 "Arduino.sch" 50
-F2 "Relay+" O R 5000 6100 60
-F3 "Relay-" I R 5000 6250 60
-F4 "MOSI" O R 5000 5050 60
-F5 "MISO" I R 5000 5250 60
-F6 "SCLK" O R 5000 5450 60
-F7 "CS_N" O R 5000 5650 60
-F8 "LED_EN" O R 5000 4300 60
-F9 "LED_FREQ" O R 5000 4500 60
-F10 "FAN_EN" I R 5000 3600 60
-F11 "TACH_MEAS" I R 5000 3800 60
+F2 "Relay+" O R 4150 6200 60
+F3 "Relay-" I R 4150 6350 60
+F4 "MOSI" O R 4150 5150 60
+F5 "MISO" I R 4150 5350 60
+F6 "SCLK" O R 4150 5550 60
+F7 "CS_N" O R 4150 5750 60
+F8 "LED_EN" O R 4150 4400 60
+F9 "LED_FREQ" O R 4150 4600 60
+F10 "FAN_EN" I R 4150 3700 60
+F11 "TACH_MEAS" I R 4150 3900 60
 $EndSheet
 $Sheet
@@
 $EndSheet
 $Sheet
-S 3400 900  1800 1450
+S 950  1000 1800 1450
 U 52ED6CD0
 F0 "Power" 50
@@
 $EndSheet
 $Sheet
-S 7600 1050 1800 1150
+S 7600 750  1800 1500
 U 52ED6D65
 F0 "Fan" 50
 F1 "Fan.sch" 50
-F2 "Power+" O R 9400 1300 60
-F3 "Power-" I R 9400 1500 60
-F4 "Tach" I R 9400 1700 60
-F5 "Tach_OUT" O L 7600 1300 60
-F6 "Fan_IN" I L 7600 1500 60
+F2 "Power+" O R 9400 1000 60
+F3 "Power-" I R 9400 1200 60
+F4 "Tach" I R 9400 1400 60
+F5 "Tach_OUT" O L 7600 950 60
+F6 "Fan_IN" I L 7600 1150 60
+F7 "Current Measure" I L 7600 1350 60
+F8 "MOSI" I L 7600 1650 60
+F9 "SLCK" I L 7600 1800 60
+F10 "CS_N" I L 7600 1950 60
+F11 "MISO" O L 7600 2100 60
 $EndSheet
 $Sheet
@@
 F1 "TerminalBlock.sch" 50
 $EndSheet
+$Sheet
+S 4250 900  2000 1650
+U 53167EEF
+F0 "PowerAdjustmentMonitor" 50
+F1 "PowerAdjustmentMonitor.sch" 50
+$EndSheet
 $EndSCHEMATC

Commit message: Week3 Part 2
Changed lines of the file:
@@
 EESchema Schematic File Version 2
+LIBS:BenchBuddy
 LIBS:power
 LIBS:device
@@
 Sheet 1 9
 Title ""
-Date "5 mar 2014"
+Date "7 mar 2014"
 Rev ""
 Comp ""
@@
 F2 "Relay+" O R 4150 6200 60
 F3 "Relay-" I R 4150 6350 60
-F4 "MOSI" O R 4150 5150 60
-F5 "MISO" I R 4150 5350 60
-F6 "SCLK" O R 4150 5550 60
-F7 "CS_N" O R 4150 5750 60
-F8 "LED_EN" O R 4150 4400 60
-F9 "LED_FREQ" O R 4150 4600 60
-F10 "FAN_EN" I R 4150 3700 60
-F11 "TACH_MEAS" I R 4150 3900 60
-$EndSheet
-$Sheet
-S 7600 4250 1800 1000
+F4 "MOSI" O R 4150 4100 60
+F5 "MISO" I R 4150 4200 60
+F6 "SCLK" O R 4150 4300 60
+F7 "TACH_MEAS" I R 4150 4600 60
+F8 "CURR_MEAS" I R 4150 4700 60
+F9 "V+_ADJ_MON" I R 4150 3400 60
+F10 "V-_ADJ_MON" I R 4150 3550 60
+F11 "LED_EN_PWM" O R 4150 5500 60
+F12 "DAC_CS_N" O R 4150 4400 60
+F13 "ADC_CS_N" O R 4150 5050 60
+F14 "FAN_PWM" I R 4150 3900 60
+F15 "FAN_MODE" O R 4150 3800 60
+$EndSheet
+$Sheet
+S 7600 4200 1800 900
 U 52ED6C3B
 F0 "Thermocoulpe" 50
 F1 "Thermocouple.sch" 50
-F2 "TC IN +" I R 9400 4400 60
-F3 "TC IN -" I R 9400 4550 60
-F4 "MOSI" I L 7600 4500 60
-F5 "MISO" O L 7600 4700 60
-F6 "SCLK" I L 7600 4900 60
-F7 "CS_N" I L 7600 5100 60
-$EndSheet
-$Sheet
-S 7600 5750 1800 1050
-U 52ED6CA1
-F0 "Relay" 50
-F1 "Relay.sch" 50
-F2 "DIN+" I L 7600 6150 60
-F3 "DIN-" O L 7600 6400 60
-F4 "Relay+" I R 9400 6150 60
-F5 "Relay-" O R 9400 6350 60
+F2 "TC IN +" I R 9400 4350 60
+F3 "TC IN -" I R 9400 4500 60
+F4 "MOSI" I L 7600 4750 60
+F5 "MISO" O L 7600 4850 60
+F6 "SCLK" I L 7600 4950 60
+F7 "CS_N" I L 7600 5050 60
 $EndSheet
 $Sheet
@@
 $EndSheet
 $Sheet
-S 7600 2700 1800 1100
+S 7600 5350 1800 700
 U 52ED6D30
 F0 "LED Driver" 50
 F1 "LED_Driver.sch" 50
-F2 "EN" I L 7600 3000 60
-F3 "FREQ" I L 7600 3200 60
-F4 "String+" O R 9400 2950 60
-F5 "String-" I R 9400 3150 60
+F2 "LED_EN_PWM" I L 7600 5500 60
+F3 "LED_String+" O R 9400 5550 60
+F4 "LED_String-" O R 9400 5800 60
 $EndSheet
 $Sheet
 S 7600 750  1800 1500
+U 53167EEF
+F0 "PowerAdjustmentMonitor" 50
+F1 "PowerAdjustmentMonitor.sch" 50
+F2 "V+_ADJ" O R 9400 1400 60
+F3 "V-_ADJ" O R 9400 1600 60
+F4 "3V3_MON" O L 7600 1500 60
+F5 "5V_MON" O L 7600 1650 60
+F6 "V+_ADJ_MON" O L 7600 1800 60
+F7 "V-_ADJ_MON" O L 7600 1950 60
+F8 "V+_CURR_MON" O L 7600 2100 60
+F9 "V-_CURR_MON" O L 7600 2200 60
+$EndSheet
+$Sheet
+S 10300 1200 750  5850
+U 52ED6DA9
+F0 "Terminal Block" 50
+F1 "TerminalBlock.sch" 50
+F2 "V+_ADJ" I L 10300 1400 60
+F3 "V-_ADJ" I L 10300 1600 60
+F4 "FAN_OUT+" O L 10300 2900 60
+F5 "FAN_OUT-" O L 10300 3050 60
+F6 "TACH_IN" I L 10300 3200 60
+F7 "LED_STRING+" O L 10300 5550 60
+F8 "LED_STRING-" O L 10300 5800 60
+F9 "TC_IN+" I L 10300 4350 60
+F10 "TC_IN-" I L 10300 4500 60
+F11 "RELAY_COM" B L 10300 6450 60
+F12 "RELAY_NO" B L 10300 6750 60
+F13 "RELAY_NC" B L 10300 6600 60
+$EndSheet
+$Sheet
+S 7600 6300 1800 750
+U 52ED6CA1
+F0 "Relay" 50
+F1 "Relay.sch" 50
+F2 "RELAY_NC" B R 9400 6600 60
+F3 "RELAY_NO" B R 9400 6750 60
+F4 "RELAY_COM" B R 9400 6450 60
+F5 "RELAY+" I L 7600 6550 60
+F6 "RELAY-" O L 7600 6650 60
+$EndSheet
+Wire Wire Line
+	9400 1400 10300 1400
+Wire Wire Line
+	10300 1600 9400 1600
+Wire Wire Line
+	9400 2900 10300 2900
+Wire Wire Line
+	10300 3050 9400 3050
+Wire Wire Line
+	9400 3200 10300 3200
+Wire Wire Line
+	10300 5550 9400 5550
+Wire Wire Line
+	9400 5800 10300 5800
+Wire Wire Line
+	10300 4350 9400 4350
+Wire Wire Line
+	9400 4500 10300 4500
+Wire Wire Line
+	10300 6450 9400 6450
+Wire Wire Line
+	9400 6600 10300 6600
+Wire Wire Line
+	10300 6750 9400 6750
+Wire Wire Line
+	4150 3400 5000 3400
+Wire Wire Line
+	5000 3400 5000 1800
+Wire Wire Line
+	5000 1800 7600 1800
+Wire Wire Line
+	4150 3550 5100 3550
+Wire Wire Line
+	5100 3550 5100 1950
+Wire Wire Line
+	5100 1950 7600 1950
+$Sheet
+S 7600 2550 1800 1400
 U 52ED6D65
 F0 "Fan" 50
 F1 "Fan.sch" 50
-F2 "Power+" O R 9400 1000 60
-F3 "Power-" I R 9400 1200 60
-F4 "Tach" I R 9400 1400 60
-F5 "Tach_OUT" O L 7600 950 60
-F6 "Fan_IN" I L 7600 1150 60
-F7 "Current Measure" I L 7600 1350 60
-F8 "MOSI" I L 7600 1650 60
-F9 "SLCK" I L 7600 1800 60
-F10 "CS_N" I L 7600 1950 60
-F11 "MISO" O L 7600 2100 60
-$EndSheet
-$Sheet
-S 10550 1200 500  5150
-U 52ED6DA9
-F0 "Terminal Block" 50
-F1 "TerminalBlock.sch" 50
-$EndSheet
-$Sheet
-S 4250 900  2000 1650
-U 53167EEF
-F0 "PowerAdjustmentMonitor" 50
-F1 "PowerAdjustmentMonitor.sch" 50
-$EndSheet
+F2 "MOSI" I L 7600 2900 60
+F3 "SLCK" I L 7600 3100 60
+F4 "CS_N" I L 7600 3200 60
+F5 "MISO" O L 7600 3000 60
+F6 "Fan_Out+" O R 9400 2900 60
+F7 "Fan_Out-" O R 9400 3050 60
+F8 "Tach_In" I R 9400 3200 60
+F9 "Tach_MEASURE" O L 7600 3650 60
+F10 "CURR_MEAS" I L 7600 3800 60
+F11 "FAN_PWM" I L 7600 2750 60
+F12 "FAN_MODE" I L 7600 2650 60
+$EndSheet
+Wire Wire Line
+	4150 3900 5400 3900
+Wire Wire Line
+	5400 3900 5400 2750
+Wire Wire Line
+	5400 2750 7600 2750
+Wire Wire Line
+	4150 4100 5500 4100
+Wire Wire Line
+	5500 2900 5500 4750
+Wire Wire Line
+	5500 2900 7600 2900
+Wire Wire Line
+	4150 4200 5600 4200
+Wire Wire Line
+	5600 4200 5600 3000
+Wire Wire Line
+	5600 3000 7600 3000
+Wire Wire Line
+	4150 4300 5700 4300
+Wire Wire Line
+	5700 4300 5700 3100
+Wire Wire Line
+	5700 3100 7600 3100
+Wire Wire Line
+	4150 4400 5800 4400
+Wire Wire Line
+	5800 4400 5800 3200
+Wire Wire Line
+	5800 3200 7600 3200
+Wire Wire Line
+	4150 4600 5900 4600
+Wire Wire Line
+	5900 4600 5900 3650
+Wire Wire Line
+	5900 3650 7600 3650
+Wire Wire Line
+	4150 4700 6000 4700
+Wire Wire Line
+	6000 4700 6000 3800
+Wire Wire Line
+	6000 3800 7600 3800
+Wire Wire Line
+	4150 5500 7600 5500
+Wire Wire Line
+	5500 4750 7600 4750
+Connection ~ 5500 4100
+Wire Wire Line
+	7600 4850 5400 4850
+Wire Wire Line
+	5400 4850 5400 4200
+Connection ~ 5400 4200
+Wire Wire Line
+	7600 4950 5300 4950
+Wire Wire Line
+	5300 4950 5300 4300
+Connection ~ 5300 4300
+Wire Wire Line
+	7600 5050 4150 5050
+Wire Wire Line
+	4150 6200 5400 6200
+Wire Wire Line
+	5400 6200 5400 6550
+Wire Wire Line
+	5400 6550 7600 6550
+Wire Wire Line
+	4150 6350 5250 6350
+Wire Wire Line
+	5250 6350 5250 6650
+Wire Wire Line
+	5250 6650 7600 6650
+Wire Wire Line
+	4150 3800 5300 3800
+Wire Wire Line
+	5300 3800 5300 2650
+Wire Wire Line
+	5300 2650 7600 2650
 $EndSCHEMATC

Commit message: Pre layout
Changed lines of the file:
@@
 Sheet 1 9
 Title ""
-Date "9 mar 2014"
+Date "30 mar 2014"
 Rev ""
 Comp ""
@@
 Comment4 ""
 $EndDescr
-$Sheet
-S 2750 3300 1400 3450
-U 52ED6BE1
-F0 "Arduino" 50
-F1 "Arduino.sch" 50
-F2 "Relay+" O R 4150 6200 60
-F3 "Relay-" I R 4150 6350 60
-F4 "MOSI" O R 4150 4100 60
-F5 "MISO" I R 4150 4200 60
-F6 "SCLK" O R 4150 4300 60
-F7 "TACH_MEAS" I R 4150 4600 60
-F8 "CURR_MEAS" I R 4150 4700 60
-F9 "V+_ADJ_MON" I R 4150 3400 60
-F10 "V-_ADJ_MON" I R 4150 3550 60
-F11 "LED_EN_PWM" O R 4150 5500 60
-F12 "DAC_CS_N" O R 4150 4400 60
-F13 "ADC_CS_N" O R 4150 5050 60
-F14 "FAN_PWM" I R 4150 3900 60
-F15 "FAN_MODE" O R 4150 3800 60
-$EndSheet
-$Sheet
-S 7600 4200 1800 900
-U 52ED6C3B
-F0 "Thermocoulpe" 50
-F1 "Thermocouple.sch" 50
-F2 "TC IN +" I R 9400 4350 60
-F3 "TC IN -" I R 9400 4500 60
-F4 "MOSI" I L 7600 4750 60
-F5 "MISO" O L 7600 4850 60
-F6 "SCLK" I L 7600 4950 60
-F7 "CS_N" I L 7600 5050 60
-$EndSheet
 $Sheet
 S 950  1000 1800 1450
@@
 F6 "V+_ADJ_MON" O L 7600 1800 60
 F7 "V-_ADJ_MON" O L 7600 1950 60
-F8 "V+_CURR_MON" O L 7600 2100 60
-F9 "V-_CURR_MON" O L 7600 2200 60
 $EndSheet
 $Sheet
@@
 	10300 6750 9400 6750
 Wire Wire Line
-	4150 3400 5000 3400
-Wire Wire Line
-	5000 3400 5000 1800
+	4150 3350 5000 3350
+Wire Wire Line
+	5000 3350 5000 1800
 Wire Wire Line
 	5000 1800 7600 1800
 Wire Wire Line
-	4150 3550 5100 3550
-Wire Wire Line
-	5100 3550 5100 1950
+	4150 3450 5100 3450
+Wire Wire Line
+	5100 3450 5100 1950
 Wire Wire Line
 	5100 1950 7600 1950
@@
 F3 "SLCK" I L 7600 3100 60
 F4 "CS_N" I L 7600 3200 60
-F5 "MISO" O L 7600 3000 60
-F6 "Fan_Out+" O R 9400 2900 60
-F7 "Fan_Out-" O R 9400 3050 60
-F8 "Tach_In" I R 9400 3200 60
-F9 "Tach_MEASURE" O L 7600 3650 60
-F10 "CURR_MEAS" I L 7600 3800 60
-F11 "FAN_PWM" I L 7600 2750 60
-F12 "FAN_MODE" I L 7600 2650 60
-$EndSheet
-Wire Wire Line
-	4150 3900 5400 3900
-Wire Wire Line
-	5400 3900 5400 2750
+F5 "Fan_Out+" O R 9400 2900 60
+F6 "Fan_Out-" O R 9400 3050 60
+F7 "Tach_In" I R 9400 3200 60
+F8 "Tach_MEASURE" O L 7600 3650 60
+F9 "CURR_MEAS" I L 7600 3800 60
+F10 "FAN_PWM" I L 7600 2750 60
+F11 "FAN_MODE" I L 7600 2650 60
+F12 "~LDAC" I L 7600 3300 60
+F13 "~SHDN" I L 7600 3400 60
+$EndSheet
+Wire Wire Line
+	4150 3750 5400 3750
+Wire Wire Line
+	5400 3750 5400 2750
 Wire Wire Line
 	5400 2750 7600 2750
 Wire Wire Line
-	4150 4100 5500 4100
-Wire Wire Line
-	5500 2900 5500 4750
+	4150 3900 5500 3900
+Wire Wire Line
+	5500 2900 5500 4500
 Wire Wire Line
 	5500 2900 7600 2900
 Wire Wire Line
-	4150 4200 5600 4200
-Wire Wire Line
-	5600 4200 5600 3000
-Wire Wire Line
-	5600 3000 7600 3000
-Wire Wire Line
-	4150 4300 5700 4300
-Wire Wire Line
-	5700 4300 5700 3100
+	4150 4100 5700 4100
+Wire Wire Line
+	5700 4100 5700 3100
 Wire Wire Line
 	5700 3100 7600 3100
 Wire Wire Line
-	4150 4400 5800 4400
-Wire Wire Line
-	5800 4400 5800 3200
+	4150 4200 5800 4200
+Wire Wire Line
+	5800 4200 5800 3200
 Wire Wire Line
 	5800 3200 7600 3200
 Wire Wire Line
-	4150 4600 5900 4600
-Wire Wire Line
-	5900 4600 5900 3650
-Wire Wire Line
-	5900 3650 7600 3650
-Wire Wire Line
-	4150 4700 6000 4700
-Wire Wire Line
-	6000 4700 6000 3800
-Wire Wire Line
-	6000 3800 7600 3800
+	4150 4450 6300 4450
+Wire Wire Line
+	6300 4450 6300 3650
+Wire Wire Line
+	6300 3650 7600 3650
+Wire Wire Line
+	4150 4550 6400 4550
+Wire Wire Line
+	6400 4550 6400 3800
+Wire Wire Line
+	6400 3800 7600 3800
 Wire Wire Line
 	4150 5500 7600 5500
 Wire Wire Line
-	5500 4750 7600 4750
-Connection ~ 5500 4100
-Wire Wire Line
-	7600 4850 5400 4850
-Wire Wire Line
-	5400 4850 5400 4200
-Connection ~ 5400 4200
-Wire Wire Line
-	7600 4950 5300 4950
-Wire Wire Line
-	5300 4950 5300 4300
-Connection ~ 5300 4300
+	5500 4500 7600 4500
+Connection ~ 5500 3900
+Wire Wire Line
+	7600 4600 5400 4600
+Wire Wire Line
+	5400 4600 5400 4000
+Wire Wire Line
+	7600 4700 5300 4700
+Wire Wire Line
+	5300 4700 5300 4100
+Connection ~ 5300 4100
 Wire Wire Line
 	7600 5050 4150 5050
@@
 	5250 6650 7600 6650
 Wire Wire Line
-	4150 3800 5300 3800
-Wire Wire Line
-	5300 3800 5300 2650
+	4150 3650 5300 3650
+Wire Wire Line
+	5300 3650 5300 2650
 Wire Wire Line
 	5300 2650 7600 2650
+$Sheet
+S 7600 4200 1800 900
+U 52ED6C3B
+F0 "Thermocoulpe" 50
+F1 "Thermocouple.sch" 50
+F2 "TC IN +" I R 9400 4350 60
+F3 "TC IN -" I R 9400 4500 60
+F4 "MOSI" I L 7600 4500 60
+F5 "MISO" O L 7600 4600 60
+F6 "SCLK" I L 7600 4700 60
+F7 "~RESET" I L 7600 4850 60
+F8 "~DR" O L 7600 4950 60
+F9 "~CS" I L 7600 5050 60
+$EndSheet
+Wire Wire Line
+	7600 4850 4150 4850
+Wire Wire Line
+	4150 4950 7600 4950
+Wire Wire Line
+	4150 4300 5900 4300
+Wire Wire Line
+	5900 4300 5900 3300
+Wire Wire Line
+	5900 3300 7600 3300
+Wire Wire Line
+	7600 3400 6000 3400
+Wire Wire Line
+	6000 3400 6000 4400
+Wire Wire Line
+	6000 4400 4150 4400
+Wire Wire Line
+	5400 4000 4150 4000
+$Sheet
+S 2750 3300 1400 3450
+U 52ED6BE1
+F0 "Arduino" 50
+F1 "Arduino.sch" 50
+F2 "Relay+" O R 4150 6200 60
+F3 "Relay-" I R 4150 6350 60
+F4 "MOSI" O R 4150 3900 60
+F5 "MISO" I R 4150 4000 60
+F6 "SCLK" O R 4150 4100 60
+F7 "TACH_MEAS" I R 4150 4450 60
+F8 "CURR_MEAS" I R 4150 4550 60
+F9 "V+_ADJ_MON" I R 4150 3350 60
+F10 "V-_ADJ_MON" I R 4150 3450 60
+F11 "LED_EN_PWM" O R 4150 5500 60
+F12 "FAN_PWM" I R 4150 3750 60
+F13 "FAN_MODE" O R 4150 3650 60
+F14 "~RESET" O R 4150 4850 60
+F15 "~DR" O R 4150 4950 60
+F16 "~LADC" I R 4150 4300 60
+F17 "~SHDN" I R 4150 4400 60
+F18 "~DAC_CS" O R 4150 4200 60
+F19 "~ADC_CS" O R 4150 5050 60
+$EndSheet
 $EndSCHEMATC
