File: BenchBuddy/PowerAdjustmentMonitor.sch (KiCad schematic (older format))
At the start: 36 parts, among them U6 LM317, U7 LM337T, U8 LM337T, U9 LM317

Commit message: Pre layout 2
Parts:
- removed U6, U9: LM317, ~, symbol LM317
- added U6, U9: LM317T, TO220_BB, symbol LM317T
- C14, C15, C16, C17, C22, C23, C24, C25: value C -> 10u
- C18, C19, C20, C21: value C -> .01u
- R36, R39: value R -> 1K
- R37, R38: value R -> 3K
- R54, R57: value R -> 9.1K
- R55, R56: value R -> 1.3K
- U7, U8: footprint TO-220 -> TO220_BB
Connections:
- net +12V: now also U6.3 (IN), U9.3 (IN)
- net -12V: now also D3.1 (A), D7.1 (A); no longer D3.2 (K), D7.2 (K)
- net FE_V+: now also U9.2 (OUT)
- net FE_V-: now also D7.2 (K); no longer D7.1 (A)
- net V+_ADJ: now also U6.2 (OUT)
- net V-_ADJ: now also D3.2 (K); no longer D3.1 (A)
- net at C19.1, D12.1 (A), R30.1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: now also U6.1 (ADJ)
- net at C20.1, D11.1 (A), R56.1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: now also U9.1 (ADJ)
Changed lines of the file:
@@
 Sheet 4 9
 Title ""
-Date "30 mar 2014"
+Date "23 apr 2014"
 Rev ""
 Comp ""
@@
 	1    4700 5450
 	-1   0    0    1
-$EndComp
-$Comp
-L LM317 U6
-U 1 1 53177EB1
-P 6900 2200
-F 0 "U6" H 6900 2500 60  0000 C CNN
-F 1 "LM317" H 6950 1950 60  0000 L CNN
-F 2 "~" H 6900 2200 60  0000 C CNN
-F 3 "~" H 6900 2200 60  0000 C CNN
-	1    6900 2200
-	1    0    0    -1
 $EndComp
 $Comp
@@
 P 8500 2550
 F 0 "R36" V 8580 2550 40  0000 C CNN
-F 1 "R" V 8507 2551 40  0000 C CNN
+F 1 "1K" V 8507 2551 40  0000 C CNN
 F 2 "~" V 8430 2550 30  0000 C CNN
 F 3 "~" H 8500 2550 30  0000 C CNN
@@
 P 8500 3550
 F 0 "R37" V 8580 3550 40  0000 C CNN
-F 1 "R" V 8507 3551 40  0000 C CNN
+F 1 "3K" V 8507 3551 40  0000 C CNN
 F 2 "~" V 8430 3550 30  0000 C CNN
 F 3 "~" H 8500 3550 30  0000 C CNN
@@
 P 8500 4400
 F 0 "R38" V 8580 4400 40  0000 C CNN
-F 1 "R" V 8507 4401 40  0000 C CNN
+F 1 "3K" V 8507 4401 40  0000 C CNN
 F 2 "~" V 8430 4400 30  0000 C CNN
 F 3 "~" H 8500 4400 30  0000 C CNN
@@
 P 8500 5350
 F 0 "R39" V 8580 5350 40  0000 C CNN
-F 1 "R" V 8507 5351 40  0000 C CNN
+F 1 "1K" V 8507 5351 40  0000 C CNN
 F 2 "~" V 8430 5350 30  0000 C CNN
 F 3 "~" H 8500 5350 30  0000 C CNN
@@
 $EndComp
 $Comp
-L LM317 U9
-U 1 1 53279B12
-P 3550 2850
-F 0 "U9" H 3550 3150 60  0000 C CNN
-F 1 "LM317" H 3600 2600 60  0000 L CNN
-F 2 "~" H 3550 2850 60  0000 C CNN
-F 3 "~" H 3550 2850 60  0000 C CNN
-	1    3550 2850
-	1    0    0    -1
-$EndComp
-$Comp
 L R R57
 U 1 1 53279B19
 P 4150 3650
 F 0 "R57" V 4230 3650 40  0000 C CNN
-F 1 "R" V 4157 3651 40  0000 C CNN
+F 1 "9.1K" V 4157 3651 40  0000 C CNN
 F 2 "~" V 4080 3650 30  0000 C CNN
 F 3 "~" H 4150 3650 30  0000 C CNN
@@
 P 4150 3050
 F 0 "R56" V 4230 3050 40  0000 C CNN
-F 1 "R" V 4157 3051 40  0000 C CNN
+F 1 "1.3K" V 4157 3051 40  0000 C CNN
 F 2 "~" V 4080 3050 30  0000 C CNN
 F 3 "~" H 4150 3050 30  0000 C CNN
@@
 F 0 "U8" H 3100 5050 40  0000 C CNN
 F 1 "LM337T" H 3300 5050 40  0000 L CNN
-F 2 "TO-220" H 3300 5150 30  0000 C CIN
+F 2 "TO220_BB" H 3300 5150 30  0000 C CIN
 F 3 "~" H 3300 5250 60  0000 C CNN
 	1    3300 5250
@@
 P 4050 4900
 F 0 "R55" V 4130 4900 40  0000 C CNN
-F 1 "R" V 4057 4901 40  0000 C CNN
+F 1 "1.3K" V 4057 4901 40  0000 C CNN
 F 2 "~" V 3980 4900 30  0000 C CNN
 F 3 "~" H 4050 4900 30  0000 C CNN
@@
 P 4050 4300
 F 0 "R54" V 4130 4300 40  0000 C CNN
-F 1 "R" V 4057 4301 40  0000 C CNN
+F 1 "9.1K" V 4057 4301 40  0000 C CNN
 F 2 "~" V 3980 4300 30  0000 C CNN
 F 3 "~" H 4050 4300 30  0000 C CNN
@@
 F 0 "U7" H 6400 5600 40  0000 C CNN
 F 1 "LM337T" H 6600 5600 40  0000 L CNN
-F 2 "TO-220" H 6600 5700 30  0000 C CIN
+F 2 "TO220_BB" H 6600 5700 30  0000 C CIN
 F 3 "~" H 6600 5800 60  0000 C CNN
 	1    6600 5800
@@
 P 7900 2950
 F 0 "C24" H 7900 3050 40  0000 L CNN
-F 1 "C" H 7906 2865 40  0000 L CNN
+F 1 "10u" H 7906 2865 40  0000 L CNN
 F 2 "~" H 7938 2800 30  0000 C CNN
 F 3 "~" H 7900 2950 60  0000 C CNN
@@
 P 4400 3350
 F 0 "C25" H 4400 3450 40  0000 L CNN
-F 1 "C" H 4406 3265 40  0000 L CNN
+F 1 "10u" H 4406 3265 40  0000 L CNN
 F 2 "~" H 4438 3200 30  0000 C CNN
 F 3 "~" H 4400 3350 60  0000 C CNN
@@
 P 4400 4600
 F 0 "C23" H 4400 4700 40  0000 L CNN
-F 1 "C" H 4406 4515 40  0000 L CNN
+F 1 "10u" H 4406 4515 40  0000 L CNN
 F 2 "~" H 4438 4450 30  0000 C CNN
 F 3 "~" H 4400 4600 60  0000 C CNN
@@
 P 7550 5150
 F 0 "C22" H 7550 5250 40  0000 L CNN
-F 1 "C" H 7556 5065 40  0000 L CNN
+F 1 "10u" H 7556 5065 40  0000 L CNN
 F 2 "~" H 7588 5000 30  0000 C CNN
 F 3 "~" H 7550 5150 60  0000 C CNN
@@
 P 6150 5150
 F 0 "C14" H 6150 5250 40  0000 L CNN
-F 1 "C" H 6156 5065 40  0000 L CNN
+F 1 "10u" H 6156 5065 40  0000 L CNN
 F 2 "~" H 6188 5000 30  0000 C CNN
 F 3 "~" H 6150 5150 60  0000 C CNN
@@
 P 2850 4500
 F 0 "C16" H 2850 4600 40  0000 L CNN
-F 1 "C" H 2856 4415 40  0000 L CNN
+F 1 "10u" H 2856 4415 40  0000 L CNN
 F 2 "~" H 2888 4350 30  0000 C CNN
 F 3 "~" H 2850 4500 60  0000 C CNN
@@
 P 2850 3350
 F 0 "C17" H 2850 3450 40  0000 L CNN
-F 1 "C" H 2856 3265 40  0000 L CNN
+F 1 "10u" H 2856 3265 40  0000 L CNN
 F 2 "~" H 2888 3200 30  0000 C CNN
 F 3 "~" H 2850 3350 60  0000 C CNN
@@
 P 6450 2950
 F 0 "C15" H 6450 3050 40  0000 L CNN
-F 1 "C" H 6456 2865 40  0000 L CNN
+F 1 "10u" H 6456 2865 40  0000 L CNN
 F 2 "~" H 6488 2800 30  0000 C CNN
 F 3 "~" H 6450 2950 60  0000 C CNN
@@
 P 3650 3650
 F 0 "C20" H 3650 3750 40  0000 L CNN
-F 1 "C" H 3656 3565 40  0000 L CNN
+F 1 ".01u" H 3656 3565 40  0000 L CNN
 F 2 "~" H 3688 3500 30  0000 C CNN
 F 3 "~" H 3650 3650 60  0000 C CNN
@@
 P 3600 4300
 F 0 "C21" H 3600 4400 40  0000 L CNN
-F 1 "C" H 3606 4215 40  0000 L CNN
+F 1 ".01u" H 3606 4215 40  0000 L CNN
 F 2 "~" H 3638 4150 30  0000 C CNN
 F 3 "~" H 3600 4300 60  0000 C CNN
@@
 P 7050 4850
 F 0 "C18" H 7050 4950 40  0000 L CNN
-F 1 "C" H 7056 4765 40  0000 L CNN
+F 1 ".01u" H 7056 4765 40  0000 L CNN
 F 2 "~" H 7088 4700 30  0000 C CNN
 F 3 "~" H 7050 4850 60  0000 C CNN
@@
 P 7150 3350
 F 0 "C19" H 7150 3450 40  0000 L CNN
-F 1 "C" H 7156 3265 40  0000 L CNN
+F 1 ".01u" H 7156 3265 40  0000 L CNN
 F 2 "~" H 7188 3200 30  0000 C CNN
 F 3 "~" H 7150 3350 60  0000 C CNN
@@
 	6900 2950 7500 2950
 Wire Wire Line
-	6900 2950 6900 2550
+	6900 2350 6900 2950
 Connection ~ 7500 2950
 Wire Wire Line
@@
 	3550 3350 4150 3350
 Wire Wire Line
-	3550 3350 3550 3200
+	3550 3000 3550 3350
 Connection ~ 4150 3350
 Wire Wire Line
@@
 F 3 "~" H 3300 5650 60  0000 C CNN
 	1    3300 5650
-	-1   0    0    1
+	1    0    0    -1
 $EndComp
 $Comp
@@
 F 3 "~" H 6600 6150 60  0000 C CNN
 	1    6600 6150
-	-1   0    0    1
+	1    0    0    -1
 $EndComp
 Wire Wire Line
@@
 	1    0    0    -1
 $EndComp
+$Comp
+L LM317T U9
+U 1 1 53580592
+P 3550 2750
+F 0 "U9" H 3350 2950 40  0000 C CNN
+F 1 "LM317T" H 3550 2950 40  0000 L CNN
+F 2 "TO220_BB" H 3550 2850 30  0000 C CIN
+F 3 "~" H 3550 2750 60  0000 C CNN
+	1    3550 2750
+	1    0    0    -1
+$EndComp
+$Comp
+L LM317T U6
+U 1 1 5358065D
+P 6900 2100
+F 0 "U6" H 6700 2300 40  0000 C CNN
+F 1 "LM317T" H 6900 2300 40  0000 L CNN
+F 2 "TO220_BB" H 6900 2200 30  0000 C CIN
+F 3 "~" H 6900 2100 60  0000 C CNN
+	1    6900 2100
+	1    0    0    -1
+$EndComp
