File: BenchBuddy/TerminalBlock.sch (KiCad schematic (older format))
At the start: 0 parts

Commit message: Pre layout
Parts:
- added P4: 12 Pin Terminal Block, symbol CONN_12
- added P5: 3 Pin Terminal Block, symbol CONN_3
Connections:
- net +3.3V: now also P4.10 (P10)
- net FAN_OUT+: now also P4.5 (P5)
- net FAN_OUT-: now also P4.4 (P4)
- net LED_STRING+: now also P4.1 (P1)
- net LED_STRING-: now also P4.2 (P2)
- net RELAY_COM: now also P5.2 (PM)
- net RELAY_NC: now also P5.3 (P3)
- net RELAY_NO: now also P5.1 (P1)
- net TACH_IN: now also P4.3 (P3)
- net TC_IN+: now also P4.6 (P6)
- net TC_IN-: now also P4.7 (P7)
- net V+_ADJ: now also P4.12 (P12)
- net V-_ADJ: now also P4.11 (P11)
- new net +5P: P4.8 (P8)
- new net GND_PWR: P4.9 (P9)
Changed lines of the file:
@@
 $Descr A4 11693 8268
 encoding utf-8
-Sheet 7 9
+Sheet 5 9
 Title ""
-Date "9 mar 2014"
+Date "30 mar 2014"
 Rev ""
 Comp ""
@@
 Comment4 ""
 $EndDescr
-Text HLabel 1400 2650 0    60   Input ~ 0
+Text HLabel 5000 4500 0    60   Input ~ 0
 V+_ADJ
-Text HLabel 1450 2950 0    60   Input ~ 0
+Text HLabel 5000 4350 0    60   Input ~ 0
 V-_ADJ
-Text HLabel 1450 3300 0    60   Output ~ 0
+Text HLabel 5000 3300 0    60   Output ~ 0
 FAN_OUT+
-Text HLabel 1450 3850 0    60   Output ~ 0
+Text HLabel 5000 3150 0    60   Output ~ 0
 FAN_OUT-
-Text HLabel 1450 4150 0    60   Input ~ 0
+Text HLabel 5000 3000 0    60   Input ~ 0
 TACH_IN
-Text HLabel 1500 4400 0    60   Output ~ 0
+Text HLabel 5000 2700 0    60   Output ~ 0
 LED_STRING+
-Text HLabel 1500 4650 0    60   Output ~ 0
+Text HLabel 5000 2850 0    60   Output ~ 0
 LED_STRING-
-Text HLabel 1500 5000 0    60   Input ~ 0
+Text HLabel 5000 3450 0    60   Input ~ 0
 TC_IN+
-Text HLabel 1450 5150 0    60   Input ~ 0
+Text HLabel 5000 3600 0    60   Input ~ 0
 TC_IN-
-Text HLabel 1450 5400 0    60   BiDi ~ 0
+Text HLabel 5000 5200 0    60   BiDi ~ 0
 RELAY_COM
-Text HLabel 1400 5600 0    60   BiDi ~ 0
+Text HLabel 5000 5050 0    60   BiDi ~ 0
 RELAY_NO
-Text HLabel 1400 5800 0    60   BiDi ~ 0
+Text HLabel 5000 5350 0    60   BiDi ~ 0
 RELAY_NC
 $Comp
-L +3,3V #PWR45
+L +3,3V #PWR032
 U 1 1 5319732A
-P 2200 1650
-F 0 "#PWR45" H 2200 1610 30  0001 C CNN
-F 1 "+3,3V" H 2200 1760 30  0000 C CNN
-F 2 "~" H 2200 1650 60  0000 C CNN
-F 3 "~" H 2200 1650 60  0000 C CNN
-	1    2200 1650
+P 4150 3900
+F 0 "#PWR032" H 4150 3860 30  0001 C CNN
+F 1 "+3,3V" H 4150 4010 30  0000 C CNN
+F 2 "~" H 4150 3900 60  0000 C CNN
+F 3 "~" H 4150 3900 60  0000 C CNN
+	1    4150 3900
 	1    0    0    -1
 $EndComp
 $Comp
-L +5V #PWR46
-U 1 1 53199BC5
-P 2450 1650
-F 0 "#PWR46" H 2450 1740 20  0001 C CNN
-F 1 "+5V" H 2450 1740 30  0000 C CNN
-F 2 "~" H 2450 1650 60  0000 C CNN
-F 3 "~" H 2450 1650 60  0000 C CNN
-	1    2450 1650
+L CONN_12 P4
+U 1 1 5324D10F
+P 7900 3650
+F 0 "P4" V 7850 3650 60  0000 C CNN
+F 1 "12 Pin Terminal Block" V 7950 3650 60  0000 C CNN
+F 2 "" H 7900 3650 60  0000 C CNN
+F 3 "" H 7900 3650 60  0000 C CNN
+F 4 "ON SHORE TECHNOLOGY INC" H 7900 3650 60  0001 C CNN "MFG Name"
+F 5 "OSTTE120104" H 7900 3650 60  0001 C CNN "MFG Part Number"
+	1    7900 3650
 	1    0    0    -1
 $EndComp
+Wire Wire Line
+	5000 2700 7350 2700
+Wire Wire Line
+	7350 2700 7350 3100
+Wire Wire Line
+	7350 3100 7550 3100
+Wire Wire Line
+	7550 3200 7250 3200
+Wire Wire Line
+	7250 3200 7250 2850
+Wire Wire Line
+	7250 2850 5000 2850
+Wire Wire Line
+	5000 3000 7150 3000
+Wire Wire Line
+	7150 3000 7150 3300
+Wire Wire Line
+	7150 3300 7550 3300
+Wire Wire Line
+	7550 3400 7050 3400
+Wire Wire Line
+	7050 3400 7050 3150
+Wire Wire Line
+	7050 3150 5000 3150
+Wire Wire Line
+	5000 3300 6950 3300
+Wire Wire Line
+	6950 3300 6950 3500
+Wire Wire Line
+	6950 3500 7550 3500
+Wire Wire Line
+	7550 3600 6850 3600
+Wire Wire Line
+	6850 3600 6850 3450
+Wire Wire Line
+	5000 3600 6750 3600
+Wire Wire Line
+	6750 3600 6750 3700
+Wire Wire Line
+	6750 3700 7550 3700
+Wire Wire Line
+	4350 3800 7550 3800
+Wire Wire Line
+	7550 3900 6750 3900
+Wire Wire Line
+	6750 3900 6750 4000
+Wire Wire Line
+	6750 4000 4350 4000
+Wire Wire Line
+	4150 4200 6850 4200
+Wire Wire Line
+	6850 4200 6850 4000
+Wire Wire Line
+	6850 4000 7550 4000
+Wire Wire Line
+	5000 4350 7000 4350
+Wire Wire Line
+	7000 4350 7000 4100
+Wire Wire Line
+	7000 4100 7550 4100
+Wire Wire Line
+	7550 4200 7100 4200
+Wire Wire Line
+	7100 4200 7100 4500
+Wire Wire Line
+	7100 4500 5000 4500
 $Comp
-L GND #PWR47
-U 1 1 53199BDE
-P 2700 1650
-F 0 "#PWR47" H 2700 1650 30  0001 C CNN
-F 1 "GND" H 2700 1580 30  0001 C CNN
-F 2 "~" H 2700 1650 60  0000 C CNN
-F 3 "~" H 2700 1650 60  0000 C CNN
-	1    2700 1650
+L CONN_3 P5
+U 1 1 5324D26F
+P 7900 5200
+F 0 "P5" V 7850 5200 50  0000 C CNN
+F 1 "3 Pin Terminal Block" V 7950 5200 40  0000 C CNN
+F 2 "" H 7900 5200 60  0000 C CNN
+F 3 "" H 7900 5200 60  0000 C CNN
+F 4 "PHOENIX CONTACT" H 7900 5200 60  0001 C CNN "MFG Name"
+F 5 "1935174" H 7900 5200 60  0001 C CNN "MFG Part Number"
+	1    7900 5200
 	1    0    0    -1
 $EndComp
+Wire Wire Line
+	7550 5200 5000 5200
+Wire Wire Line
+	5200 5050 5200 5100
+Wire Wire Line
+	5200 5100 7550 5100
+Wire Wire Line
+	5200 5050 5000 5050
+Wire Wire Line
+	5000 5350 5200 5350
+Wire Wire Line
+	5200 5350 5200 5300
+Wire Wire Line
+	5200 5300 7550 5300
+Wire Wire Line
+	6850 3450 5000 3450
+Wire Wire Line
+	4150 4200 4150 3900
+$Comp
+L GND_PWR #PWR033
+U 1 1 53372B75
+P 4350 4100
+F 0 "#PWR033" H 4350 4100 30  0001 C CNN
+F 1 "GND_PWR" H 4350 4030 30  0000 C CNN
+F 2 "~" H 4350 4100 60  0000 C CNN
+F 3 "~" H 4350 4100 60  0000 C CNN
+	1    4350 4100
+	1    0    0    -1
+$EndComp
+Wire Wire Line
+	4350 4000 4350 4100
+Wire Wire Line
+	4350 3650 4350 3800
+$Comp
+L +5P #PWR37
+U 1 1 533748FF
+P 4350 3650
+F 0 "#PWR37" H 4350 3780 20  0001 C CNN
+F 1 "+5P" H 4350 3750 30  0000 C CNN
+F 2 "~" H 4350 3650 60  0000 C CNN
+F 3 "~" H 4350 3650 60  0000 C CNN
+	1    4350 3650
+	1    0    0    -1
+$EndComp

Commit message: Pre layout 2
Parts:
- added C26, C27, C28, C29: 10u, SM1210, symbol C
- added R34: 0, SM0805, symbol R
Connections:
- net +3.3V: now also C27.1
- net +5P: now also C26.1
- net GND_PWR: now also C26.2
- net TACH_IN: now also R34.1
- net V+_ADJ: now also C29.1
- net V-_ADJ: now also C28.1
Other:
- moved on the sheet: P5
Changed lines of the file:
@@
 Sheet 5 9
 Title ""
-Date "30 mar 2014"
+Date "23 apr 2014"
 Rev ""
 Comp ""
@@
 Comment4 ""
 $EndDescr
-Text HLabel 5000 4500 0    60   Input ~ 0
+Text HLabel 4350 4500 0    60   Input ~ 0
 V+_ADJ
-Text HLabel 5000 4350 0    60   Input ~ 0
+Text HLabel 4350 4350 0    60   Input ~ 0
 V-_ADJ
-Text HLabel 5000 3300 0    60   Output ~ 0
+Text HLabel 4350 3300 0    60   Output ~ 0
 FAN_OUT+
-Text HLabel 5000 3150 0    60   Output ~ 0
+Text HLabel 4350 3150 0    60   Output ~ 0
 FAN_OUT-
-Text HLabel 5000 3000 0    60   Input ~ 0
+Text HLabel 4350 3000 0    60   Input ~ 0
 TACH_IN
-Text HLabel 5000 2700 0    60   Output ~ 0
+Text HLabel 4350 2700 0    60   Output ~ 0
 LED_STRING+
-Text HLabel 5000 2850 0    60   Output ~ 0
+Text HLabel 4350 2850 0    60   Output ~ 0
 LED_STRING-
-Text HLabel 5000 3450 0    60   Input ~ 0
+Text HLabel 4350 3450 0    60   Input ~ 0
 TC_IN+
-Text HLabel 5000 3600 0    60   Input ~ 0
+Text HLabel 4350 3600 0    60   Input ~ 0
 TC_IN-
-Text HLabel 5000 5200 0    60   BiDi ~ 0
+Text HLabel 4350 5900 0    60   BiDi ~ 0
 RELAY_COM
-Text HLabel 5000 5050 0    60   BiDi ~ 0
+Text HLabel 4350 5750 0    60   BiDi ~ 0
 RELAY_NO
-Text HLabel 5000 5350 0    60   BiDi ~ 0
+Text HLabel 4350 6050 0    60   BiDi ~ 0
 RELAY_NC
 $Comp
 L +3,3V #PWR032
 U 1 1 5319732A
-P 4150 3900
-F 0 "#PWR032" H 4150 3860 30  0001 C CNN
-F 1 "+3,3V" H 4150 4010 30  0000 C CNN
-F 2 "~" H 4150 3900 60  0000 C CNN
-F 3 "~" H 4150 3900 60  0000 C CNN
-	1    4150 3900
+P 3500 3900
+F 0 "#PWR032" H 3500 3860 30  0001 C CNN
+F 1 "+3,3V" H 3500 4010 30  0000 C CNN
+F 2 "~" H 3500 3900 60  0000 C CNN
+F 3 "~" H 3500 3900 60  0000 C CNN
+	1    3500 3900
 	1    0    0    -1
 $EndComp
@@
 	1    0    0    -1
 $EndComp
-Wire Wire Line
-	5000 2700 7350 2700
-Wire Wire Line
-	7350 2700 7350 3100
-Wire Wire Line
-	7350 3100 7550 3100
-Wire Wire Line
-	7550 3200 7250 3200
-Wire Wire Line
-	7250 3200 7250 2850
-Wire Wire Line
-	7250 2850 5000 2850
-Wire Wire Line
-	5000 3000 7150 3000
-Wire Wire Line
-	7150 3000 7150 3300
-Wire Wire Line
-	7150 3300 7550 3300
-Wire Wire Line
-	7550 3400 7050 3400
-Wire Wire Line
-	7050 3400 7050 3150
-Wire Wire Line
-	7050 3150 5000 3150
-Wire Wire Line
-	5000 3300 6950 3300
-Wire Wire Line
-	6950 3300 6950 3500
-Wire Wire Line
-	6950 3500 7550 3500
-Wire Wire Line
-	7550 3600 6850 3600
-Wire Wire Line
-	6850 3600 6850 3450
-Wire Wire Line
-	5000 3600 6750 3600
-Wire Wire Line
-	6750 3600 6750 3700
-Wire Wire Line
-	6750 3700 7550 3700
-Wire Wire Line
-	4350 3800 7550 3800
-Wire Wire Line
-	7550 3900 6750 3900
-Wire Wire Line
-	6750 3900 6750 4000
-Wire Wire Line
-	6750 4000 4350 4000
-Wire Wire Line
-	4150 4200 6850 4200
-Wire Wire Line
-	6850 4200 6850 4000
-Wire Wire Line
-	6850 4000 7550 4000
-Wire Wire Line
-	5000 4350 7000 4350
-Wire Wire Line
-	7000 4350 7000 4100
-Wire Wire Line
-	7000 4100 7550 4100
-Wire Wire Line
-	7550 4200 7100 4200
-Wire Wire Line
-	7100 4200 7100 4500
-Wire Wire Line
-	7100 4500 5000 4500
 $Comp
 L CONN_3 P5
 U 1 1 5324D26F
-P 7900 5200
-F 0 "P5" V 7850 5200 50  0000 C CNN
-F 1 "3 Pin Terminal Block" V 7950 5200 40  0000 C CNN
-F 2 "" H 7900 5200 60  0000 C CNN
-F 3 "" H 7900 5200 60  0000 C CNN
-F 4 "PHOENIX CONTACT" H 7900 5200 60  0001 C CNN "MFG Name"
-F 5 "1935174" H 7900 5200 60  0001 C CNN "MFG Part Number"
-	1    7900 5200
-	1    0    0    -1
-$EndComp
-Wire Wire Line
-	7550 5200 5000 5200
-Wire Wire Line
-	5200 5050 5200 5100
-Wire Wire Line
-	5200 5100 7550 5100
-Wire Wire Line
-	5200 5050 5000 5050
-Wire Wire Line
-	5000 5350 5200 5350
-Wire Wire Line
-	5200 5350 5200 5300
-Wire Wire Line
-	5200 5300 7550 5300
-Wire Wire Line
-	6850 3450 5000 3450
-Wire Wire Line
-	4150 4200 4150 3900
+P 7900 5900
+F 0 "P5" V 7850 5900 50  0000 C CNN
+F 1 "3 Pin Terminal Block" V 7950 5900 40  0000 C CNN
+F 2 "" H 7900 5900 60  0000 C CNN
+F 3 "" H 7900 5900 60  0000 C CNN
+F 4 "PHOENIX CONTACT" H 7900 5900 60  0001 C CNN "MFG Name"
+F 5 "1935174" H 7900 5900 60  0001 C CNN "MFG Part Number"
+	1    7900 5900
+	1    0    0    -1
+$EndComp
 $Comp
 L GND_PWR #PWR033
 U 1 1 53372B75
-P 4350 4100
-F 0 "#PWR033" H 4350 4100 30  0001 C CNN
-F 1 "GND_PWR" H 4350 4030 30  0000 C CNN
-F 2 "~" H 4350 4100 60  0000 C CNN
-F 3 "~" H 4350 4100 60  0000 C CNN
-	1    4350 4100
-	1    0    0    -1
-$EndComp
-Wire Wire Line
-	4350 4000 4350 4100
-Wire Wire Line
-	4350 3650 4350 3800
+P 3700 4100
+F 0 "#PWR033" H 3700 4100 30  0001 C CNN
+F 1 "GND_PWR" H 3700 4030 30  0000 C CNN
+F 2 "~" H 3700 4100 60  0000 C CNN
+F 3 "~" H 3700 4100 60  0000 C CNN
+	1    3700 4100
+	1    0    0    -1
+$EndComp
 $Comp
 L +5P #PWR37
 U 1 1 533748FF
-P 4350 3650
-F 0 "#PWR37" H 4350 3780 20  0001 C CNN
-F 1 "+5P" H 4350 3750 30  0000 C CNN
-F 2 "~" H 4350 3650 60  0000 C CNN
-F 3 "~" H 4350 3650 60  0000 C CNN
-	1    4350 3650
-	1    0    0    -1
-$EndComp
+P 3700 3650
+F 0 "#PWR37" H 3700 3780 20  0001 C CNN
+F 1 "+5P" H 3700 3750 30  0000 C CNN
+F 2 "~" H 3700 3650 60  0000 C CNN
+F 3 "~" H 3700 3650 60  0000 C CNN
+	1    3700 3650
+	1    0    0    -1
+$EndComp
+$Comp
+L R R34
+U 1 1 533971FF
+P 6450 5000
+F 0 "R34" V 6530 5000 40  0000 C CNN
+F 1 "0" V 6457 5001 40  0000 C CNN
+F 2 "SM0805" V 6380 5000 30  0000 C CNN
+F 3 "~" H 6450 5000 30  0000 C CNN
+	1    6450 5000
+	1    0    0    -1
+$EndComp
+$Comp
+L GND_PWR #PWR034
+U 1 1 5339720C
+P 6650 5400
+F 0 "#PWR034" H 6650 5400 30  0001 C CNN
+F 1 "GND_PWR" H 6650 5330 30  0000 C CNN
+F 2 "~" H 6650 5400 60  0000 C CNN
+F 3 "~" H 6650 5400 60  0000 C CNN
+	1    6650 5400
+	1    0    0    -1
+$EndComp
+$Comp
+L C C29
+U 1 1 53397254
+P 6150 5050
+F 0 "C29" H 6150 5150 40  0000 L CNN
+F 1 "10u" H 6156 4965 40  0000 L CNN
+F 2 "SM1210 " H 6188 4900 30  0000 C CNN
+F 3 "~" H 6150 5050 60  0000 C CNN
+	1    6150 5050
+	1    0    0    -1
+$EndComp
+$Comp
+L C C28
+U 1 1 53397274
+P 5850 5050
+F 0 "C28" H 5850 5150 40  0000 L CNN
+F 1 "10u" H 5856 4965 40  0000 L CNN
+F 2 "SM1210 " H 5888 4900 30  0000 C CNN
+F 3 "~" H 5850 5050 60  0000 C CNN
+	1    5850 5050
+	1    0    0    -1
+$EndComp
+$Comp
+L C C27
+U 1 1 5339727A
+P 5550 5050
+F 0 "C27" H 5550 5150 40  0000 L CNN
+F 1 "10u" H 5556 4965 40  0000 L CNN
+F 2 "SM1210 " H 5588 4900 30  0000 C CNN
+F 3 "~" H 5550 5050 60  0000 C CNN
+	1    5550 5050
+	1    0    0    -1
+$EndComp
+$Comp
+L C C26
+U 1 1 53397280
+P 5250 5050
+F 0 "C26" H 5250 5150 40  0000 L CNN
+F 1 "10u" H 5256 4965 40  0000 L CNN
+F 2 "SM1210 " H 5288 4900 30  0000 C CNN
+F 3 "~" H 5250 5050 60  0000 C CNN
+	1    5250 5050
+	1    0    0    -1
+$EndComp
+Wire Wire Line
+	4350 2700 7350 2700
+Wire Wire Line
+	7350 2700 7350 3100
+Wire Wire Line
+	7350 3100 7550 3100
+Wire Wire Line
+	7550 3200 7250 3200
+Wire Wire Line
+	7250 3200 7250 2850
+Wire Wire Line
+	7250 2850 4350 2850
+Wire Wire Line
+	4350 3000 7150 3000
+Wire Wire Line
+	7150 3000 7150 3300
+Wire Wire Line
+	7150 3300 7550 3300
+Wire Wire Line
+	7550 3400 7050 3400
+Wire Wire Line
+	7050 3400 7050 3150
+Wire Wire Line
+	7050 3150 4350 3150
+Wire Wire Line
+	4350 3300 6950 3300
+Wire Wire Line
+	6950 3300 6950 3500
+Wire Wire Line
+	6950 3500 7550 3500
+Wire Wire Line
+	7550 3600 6850 3600
+Wire Wire Line
+	6850 3600 6850 3450
+Wire Wire Line
+	4350 3600 6750 3600
+Wire Wire Line
+	6750 3600 6750 3700
+Wire Wire Line
+	6750 3700 7550 3700
+Wire Wire Line
+	3700 3800 7550 3800
+Wire Wire Line
+	7550 3900 6750 3900
+Wire Wire Line
+	6750 3900 6750 4000
+Wire Wire Line
+	6750 4000 3700 4000
+Wire Wire Line
+	3500 4200 6850 4200
+Wire Wire Line
+	6850 4200 6850 4000
+Wire Wire Line
+	6850 4000 7550 4000
+Wire Wire Line
+	4350 4350 7000 4350
+Wire Wire Line
+	7000 4350 7000 4100
+Wire Wire Line
+	7000 4100 7550 4100
+Wire Wire Line
+	7550 4200 7100 4200
+Wire Wire Line
+	7100 4200 7100 4500
+Wire Wire Line
+	7100 4500 4350 4500
+Wire Wire Line
+	7550 5900 4350 5900
+Wire Wire Line
+	5200 5750 5200 5800
+Wire Wire Line
+	5200 5800 7550 5800
+Wire Wire Line
+	5200 5750 4350 5750
+Wire Wire Line
+	4350 6050 5200 6050
+Wire Wire Line
+	5200 6050 5200 6000
+Wire Wire Line
+	5200 6000 7550 6000
+Wire Wire Line
+	6850 3450 4350 3450
+Wire Wire Line
+	3500 4200 3500 3900
+Wire Wire Line
+	3700 4000 3700 4100
+Wire Wire Line
+	3700 3650 3700 3800
+Wire Wire Line
+	6650 5400 6650 5250
+Wire Wire Line
+	6650 5250 5250 5250
+Wire Wire Line
+	5250 4850 5250 3800
+Connection ~ 5250 3800
+Wire Wire Line
+	5550 4850 5550 4200
+Connection ~ 5550 4200
+Wire Wire Line
+	5850 4850 5850 4350
+Connection ~ 5850 4350
+Wire Wire Line
+	6150 4850 6150 4500
+Connection ~ 6150 4500
+Wire Wire Line
+	6450 4750 6450 3000
+Connection ~ 6450 3000
 $EndSCHEMATC
