File: BenchBuddy/Thermocouple.sch (KiCad schematic (older format))
At the start: 23 parts, among them P2 CONN_3X2, P3 CONN_2, U2 MCP3901, U3 LMT84, U4 OPA4170

Commit message: Pre layout 2
Parts:
- added C30, C31: NoPop, SM0805, symbol C
- C1: value C -> 100PF
- C10, C6, C7, C8, C9: value C -> 1u
- L5: value INDUCTOR -> 1u
- R21, R22, R25, R27: value R -> 5K
- R23, R24: value R -> 200K
- R42: value R -> 10
- R43: value R -> 100
- R44: value R -> 1000
Connections:
- net REF- is gone; now on net AGND: U2.10 (REFIN-)
- net AGND: now also C31.1
- net at U2.15 (OSC1): now also C30.1
- net at U2.16 (OSC2): now also C30.2
- net REF+: no longer names the net of U2.9 (REFIN/OUT+)
- net REF+: now also C31.2
Changed lines of the file:
@@
 Sheet 8 9
 Title ""
-Date "30 mar 2014"
+Date "23 apr 2014"
 Rev ""
 Comp ""
@@
 P 6600 3750
 F 0 "C1" H 6600 3850 40  0000 L CNN
-F 1 "C" H 6606 3665 40  0000 L CNN
+F 1 "100PF" H 6606 3665 40  0000 L CNN
 F 2 "~" H 6638 3600 30  0000 C CNN
 F 3 "~" H 6600 3750 60  0000 C CNN
@@
 P 8600 2700
 F 0 "R25" V 8680 2700 40  0000 C CNN
-F 1 "R" V 8607 2701 40  0000 C CNN
+F 1 "5K" V 8607 2701 40  0000 C CNN
 F 2 "~" V 8530 2700 30  0000 C CNN
 F 3 "~" H 8600 2700 30  0000 C CNN
@@
 P 8600 4100
 F 0 "R27" V 8680 4100 40  0000 C CNN
-F 1 "R" V 8607 4101 40  0000 C CNN
+F 1 "5K" V 8607 4101 40  0000 C CNN
 F 2 "~" V 8530 4100 30  0000 C CNN
 F 3 "~" H 8600 4100 30  0000 C CNN
@@
 P 8050 2350
 F 0 "R23" V 8130 2350 40  0000 C CNN
-F 1 "R" V 8057 2351 40  0000 C CNN
+F 1 "200K" V 8057 2351 40  0000 C CNN
 F 2 "~" V 7980 2350 30  0000 C CNN
 F 3 "~" H 8050 2350 30  0000 C CNN
@@
 P 6950 2350
 F 0 "R22" V 7030 2350 40  0000 C CNN
-F 1 "R" V 6957 2351 40  0000 C CNN
+F 1 "5K" V 6957 2351 40  0000 C CNN
 F 2 "~" V 6880 2350 30  0000 C CNN
 F 3 "~" H 6950 2350 30  0000 C CNN
@@
 P 6900 4450
 F 0 "R21" V 6980 4450 40  0000 C CNN
-F 1 "R" V 6907 4451 40  0000 C CNN
+F 1 "5K" V 6907 4451 40  0000 C CNN
 F 2 "~" V 6830 4450 30  0000 C CNN
 F 3 "~" H 6900 4450 30  0000 C CNN
@@
 P 8050 4450
 F 0 "R24" V 8130 4450 40  0000 C CNN
-F 1 "R" V 8057 4451 40  0000 C CNN
+F 1 "200K" V 8057 4451 40  0000 C CNN
 F 2 "~" V 7980 4450 30  0000 C CNN
 F 3 "~" H 8050 4450 30  0000 C CNN
@@
 Text Notes 7650 1700 0    60   ~ 0
 Instrumentation Amp
-Text Notes 1950 2700 0    60   ~ 0
+Text Notes 1900 2600 0    60   ~ 0
 16/24Bit ADC
 $Comp
@@
 P 10350 3750
 F 0 "R42" V 10430 3750 40  0000 C CNN
-F 1 "R" V 10357 3751 40  0000 C CNN
+F 1 "10" V 10357 3751 40  0000 C CNN
 F 2 "~" V 10280 3750 30  0000 C CNN
 F 3 "~" H 10350 3750 30  0000 C CNN
@@
 P 10550 3750
 F 0 "R43" V 10630 3750 40  0000 C CNN
-F 1 "R" V 10557 3751 40  0000 C CNN
+F 1 "100" V 10557 3751 40  0000 C CNN
 F 2 "~" V 10480 3750 30  0000 C CNN
 F 3 "~" H 10550 3750 30  0000 C CNN
@@
 P 10750 3750
 F 0 "R44" V 10830 3750 40  0000 C CNN
-F 1 "R" V 10757 3751 40  0000 C CNN
+F 1 "1000" V 10757 3751 40  0000 C CNN
 F 2 "~" V 10680 3750 30  0000 C CNN
 F 3 "~" H 10750 3750 30  0000 C CNN
@@
 Connection ~ 5850 6400
 $Comp
-L +5V #PWR044
+L +5V #PWR045
 U 1 1 5321056E
 P 6350 4900
-F 0 "#PWR044" H 6350 4990 20  0001 C CNN
+F 0 "#PWR045" H 6350 4990 20  0001 C CNN
 F 1 "+5V" H 6350 4990 30  0000 C CNN
 F 2 "~" H 6350 4900 60  0000 C CNN
@@
 P 7050 5650
 F 0 "C8" H 7050 5750 40  0000 L CNN
-F 1 "C" H 7056 5565 40  0000 L CNN
+F 1 "1u" H 7056 5565 40  0000 L CNN
 F 2 "~" H 7088 5500 30  0000 C CNN
 F 3 "~" H 7050 5650 60  0000 C CNN
@@
 P 7500 4050
 F 0 "C10" H 7500 4150 40  0000 L CNN
-F 1 "C" H 7506 3965 40  0000 L CNN
+F 1 "1u" H 7506 3965 40  0000 L CNN
 F 2 "~" H 7538 3900 30  0000 C CNN
 F 3 "~" H 7500 4050 60  0000 C CNN
@@
 P 7500 2900
 F 0 "C9" H 7500 3000 40  0000 L CNN
-F 1 "C" H 7506 2815 40  0000 L CNN
+F 1 "1u" H 7506 2815 40  0000 L CNN
 F 2 "~" H 7538 2750 30  0000 C CNN
 F 3 "~" H 7500 2900 60  0000 C CNN
@@
 Connection ~ 7250 2700
 $Comp
-L +5V #PWR045
+L +5V #PWR046
 U 1 1 53210982
 P 4000 1850
-F 0 "#PWR045" H 4000 1940 20  0001 C CNN
+F 0 "#PWR046" H 4000 1940 20  0001 C CNN
 F 1 "+5V" H 4000 1940 30  0000 C CNN
 F 2 "~" H 4000 1850 60  0000 C CNN
@@
 Wire Wire Line
 	4000 1850 4000 2300
-Text GLabel 5200 2900 2    60   Input ~ 0
-REF+
-Text GLabel 5200 3050 2    60   Input ~ 0
-REF-
 $Comp
 L C C7
@@
 P 4600 2150
 F 0 "C7" H 4600 2250 40  0000 L CNN
-F 1 "C" H 4606 2065 40  0000 L CNN
+F 1 "1u" H 4606 2065 40  0000 L CNN
 F 2 "~" H 4638 2000 30  0000 C CNN
 F 3 "~" H 4600 2150 60  0000 C CNN
@@
 P 2900 2150
 F 0 "C6" H 2900 2250 40  0000 L CNN
-F 1 "C" H 2906 2065 40  0000 L CNN
+F 1 "1u" H 2906 2065 40  0000 L CNN
 F 2 "~" H 2938 2000 30  0000 C CNN
 F 3 "~" H 2900 2150 60  0000 C CNN
@@
 	5400 5050 5400 6400
 Wire Wire Line
-	5200 2900 4900 2900
-Wire Wire Line
-	4900 3050 5200 3050
-$Comp
-L FE_V- #PWR58
+	4900 2900 5350 2900
+Wire Wire Line
+	4900 3050 5350 3050
+$Comp
+L FE_V- #PWR60
 U 1 1 532F3D09
 P 7250 2600
-F 0 "#PWR58" H 7250 2800 40  0001 C CNN
+F 0 "#PWR60" H 7250 2800 40  0001 C CNN
 F 1 "FE_V-" H 7250 2750 40  0000 C CNN
 F 2 "~" H 7250 2600 60  0000 C CNN
@@
 $EndComp
 $Comp
-L FE_V+ #PWR046
+L FE_V+ #PWR047
 U 1 1 532F3D22
 P 7250 3900
-F 0 "#PWR046" H 7250 4000 30  0001 C CNN
+F 0 "#PWR047" H 7250 4000 30  0001 C CNN
 F 1 "FE_V+" H 7250 4000 30  0000 C CNN
 F 2 "~" H 7250 3900 60  0000 C CNN
@@
 $EndComp
 $Comp
-L FE_V- #PWR64
+L FE_V- #PWR66
 U 1 1 532F3D39
 P 9450 3950
-F 0 "#PWR64" H 9450 4150 40  0001 C CNN
+F 0 "#PWR66" H 9450 4150 40  0001 C CNN
 F 1 "FE_V-" H 9450 4100 40  0000 C CNN
 F 2 "~" H 9450 3950 60  0000 C CNN
@@
 $EndComp
 $Comp
-L FE_V+ #PWR047
+L FE_V+ #PWR048
 U 1 1 532F3D3F
 P 9450 4950
-F 0 "#PWR047" H 9450 5050 30  0001 C CNN
+F 0 "#PWR048" H 9450 5050 30  0001 C CNN
 F 1 "FE_V+" H 9450 5050 30  0000 C CNN
 F 2 "~" H 9450 4950 60  0000 C CNN
@@
 $EndComp
 $Comp
-L FE_V+ #PWR048
+L FE_V+ #PWR049
 U 1 1 532F3D45
 P 9450 1850
-F 0 "#PWR048" H 9450 1950 30  0001 C CNN
+F 0 "#PWR049" H 9450 1950 30  0001 C CNN
 F 1 "FE_V+" H 9450 1950 30  0000 C CNN
 F 2 "~" H 9450 1850 60  0000 C CNN
@@
 $EndComp
 $Comp
-L FE_V- #PWR63
+L FE_V- #PWR65
 U 1 1 532F3D4B
 P 9450 2850
-F 0 "#PWR63" H 9450 3050 40  0001 C CNN
+F 0 "#PWR65" H 9450 3050 40  0001 C CNN
 F 1 "FE_V-" H 9450 3000 40  0000 C CNN
 F 2 "~" H 9450 2850 60  0000 C CNN
@@
 $EndComp
 $Comp
-L AGND #PWR049
+L AGND #PWR050
 U 1 1 533721EE
 P 3500 5050
-F 0 "#PWR049" H 3500 5050 40  0001 C CNN
+F 0 "#PWR050" H 3500 5050 40  0001 C CNN
 F 1 "AGND" H 3500 4980 50  0000 C CNN
 F 2 "~" H 3500 5050 60  0000 C CNN
@@
 $EndComp
 $Comp
-L AGND #PWR050
+L AGND #PWR051
 U 1 1 533721FB
 P 4000 5050
-F 0 "#PWR050" H 4000 5050 40  0001 C CNN
+F 0 "#PWR051" H 4000 5050 40  0001 C CNN
 F 1 "AGND" H 4000 4980 50  0000 C CNN
 F 2 "~" H 4000 5050 60  0000 C CNN
@@
 $EndComp
 $Comp
-L AGND #PWR051
+L AGND #PWR052
 U 1 1 53372201
 P 2550 2350
-F 0 "#PWR051" H 2550 2350 40  0001 C CNN
+F 0 "#PWR052" H 2550 2350 40  0001 C CNN
 F 1 "AGND" H 2550 2280 50  0000 C CNN
 F 2 "~" H 2550 2350 60  0000 C CNN
@@
 $EndComp
 $Comp
-L AGND #PWR052
+L AGND #PWR053
 U 1 1 53372216
 P 4950 2350
-F 0 "#PWR052" H 4950 2350 40  0001 C CNN
+F 0 "#PWR053" H 4950 2350 40  0001 C CNN
 F 1 "AGND" H 4950 2280 50  0000 C CNN
 F 2 "~" H 4950 2350 60  0000 C CNN
@@
 $EndComp
 $Comp
-L AGND #PWR053
+L AGND #PWR054
 U 1 1 5337221C
 P 7500 3150
-F 0 "#PWR053" H 7500 3150 40  0001 C CNN
+F 0 "#PWR054" H 7500 3150 40  0001 C CNN
 F 1 "AGND" H 7500 3080 50  0000 C CNN
 F 2 "~" H 7500 3150 60  0000 C CNN
@@
 $EndComp
 $Comp
-L AGND #PWR054
+L AGND #PWR055
 U 1 1 5337222C
 P 7500 4300
-F 0 "#PWR054" H 7500 4300 40  0001 C CNN
+F 0 "#PWR055" H 7500 4300 40  0001 C CNN
 F 1 "AGND" H 7500 4230 50  0000 C CNN
 F 2 "~" H 7500 4300 60  0000 C CNN
@@
 $EndComp
 $Comp
-L AGND #PWR055
+L AGND #PWR056
 U 1 1 53372232
 P 6550 4600
-F 0 "#PWR055" H 6550 4600 40  0001 C CNN
+F 0 "#PWR056" H 6550 4600 40  0001 C CNN
 F 1 "AGND" H 6550 4530 50  0000 C CNN
 F 2 "~" H 6550 4600 60  0000 C CNN
@@
 $EndComp
 $Comp
-L AGND #PWR056
+L AGND #PWR057
 U 1 1 53372238
 P 5850 6550
-F 0 "#PWR056" H 5850 6550 40  0001 C CNN
+F 0 "#PWR057" H 5850 6550 40  0001 C CNN
 F 1 "AGND" H 5850 6480 50  0000 C CNN
 F 2 "~" H 5850 6550 60  0000 C CNN
@@
 P 3700 1950
 F 0 "L5" V 3650 1950 40  0000 C CNN
-F 1 "INDUCTOR" V 3800 1950 40  0000 C CNN
+F 1 "1u" V 3800 1950 40  0000 C CNN
 F 2 "SM0805" V 3900 1950 60  0000 C CNN
 F 3 "~" H 3700 1950 60  0000 C CNN
@@
 $EndComp
 Wire Wire Line
-	3500 2150 3100 2150
+	3100 2150 3500 2150
 Wire Wire Line
 	3400 1950 3400 2150
 Connection ~ 3400 2150
+$Comp
+L C C30
+U 1 1 53401C41
+P 2300 2850
+F 0 "C30" H 2300 2950 40  0000 L CNN
+F 1 "NoPop" H 2306 2765 40  0000 L CNN
+F 2 "SM0805" H 2338 2700 30  0000 C CNN
+F 3 "~" H 2300 2850 60  0000 C CNN
+	1    2300 2850
+	-1   0    0    -1
+$EndComp
+Wire Wire Line
+	2300 2650 2500 2650
+Wire Wire Line
+	2500 2650 2500 2800
+Wire Wire Line
+	2500 2800 2750 2800
+Wire Wire Line
+	2750 2950 2500 2950
+Wire Wire Line
+	2500 2950 2500 3050
+Wire Wire Line
+	2500 3050 2300 3050
+$Comp
+L C C31
+U 1 1 53401D2A
+P 5550 2950
+F 0 "C31" H 5550 3050 40  0000 L CNN
+F 1 "NoPop" H 5556 2865 40  0000 L CNN
+F 2 "SM0805" H 5588 2800 30  0000 C CNN
+F 3 "~" H 5550 2950 60  0000 C CNN
+	1    5550 2950
+	-1   0    0    1
+$EndComp
+Wire Wire Line
+	5550 2750 5350 2750
+Wire Wire Line
+	5350 2750 5350 2900
+Wire Wire Line
+	5350 3050 5350 3150
+Wire Wire Line
+	5350 3150 5550 3150
+$Comp
+L AGND #PWR058
+U 1 1 534021A2
+P 5450 3200
+F 0 "#PWR058" H 5450 3200 40  0001 C CNN
+F 1 "AGND" H 5450 3130 50  0000 C CNN
+F 2 "~" H 5450 3200 60  0000 C CNN
+F 3 "~" H 5450 3200 60  0000 C CNN
+	1    5450 3200
+	1    0    0    -1
+$EndComp
+Wire Wire Line
+	5450 3200 5450 3150
+Connection ~ 5450 3150
 $EndSCHEMATC
